File: KiCad/MOMI.kicad_pcb (KiCad board)
At the start: 2 copper layers, 69.8 x 69.8 mm, 58 parts, among them J1 Conn_02x04_Male, J10 Conn_01x05_Male, J11 AudioJack4, J12 Conn_01x04_Female, J13 Dual Footswitch, J2 MIDI in, J3 Conn_02x04_Male, J4 MIDI out, J5 JST 1mm (I2C), J6 USB_A, J7 Conn_01x18_Female, J8 Conn_01x18_Female, J9 Expression Pedal, SW1 Encoder_Switch, SW2 SW_SPDT, U1 6N137, U2 MAX1555EZK_T

Commit message: Add KiCad files
Parts:
- removed the R12 at (111.8, 102.2)
- removed R13, R14: 10k, R_SMD_3D:R_0805_2012Metric
- added J14: Conn_01x03_Male, Pin_Headers:Pin_Header_Straight_1x03_Pitch2.54mm, F.Cu at (103.8, 119.0)
- D1: footprint D_SMD_3D:D_0805_2012Metric -> Diodes_ThroughHole:D_A-405_P2.54mm_Vertical_AnodeUp
- D2: value LED -> Green LED
- D3, D4, D8: value LED -> Red LED
- D5: renamed from D7; value LED -> Green LED
- D6: renamed from D5; value LED -> Red LED
- D7: renamed from D6; value LED -> Blue LED
- J2, J4: footprint Connect:SDS-50J -> Conn_Aud_3D:SDS-50J
- U1: value 6N137 -> H11L1M; footprint Housings_DIP:DIP-8_W7.62mm_Socket -> digikey-footprints:DIP-6_W7.62mm
- moved D1 3.98 mm to (111.7, 120.6)
- moved R2 3.76 mm to (111.7, 117.9), turned to 0 degrees
- moved U1 3.16 mm to (114.7, 118.6)
- moved R1 2.70 mm to (124.5, 118.7)
- moved C1 0.76 mm to (108.7, 130.2)
- moved R16 0.57 mm to (105.3, 130.2)
- moved J6 0.44 mm to (100.1, 119.0)
- renumbered C5 to C2, C2 to C3, C6 to C4, C3 to C5, C4 to C6, J9 to J10, J10 to J11, J11 to J12, J12 to J7, J7 to J8, J8 to J9, R21 to R11, R11 to R12, R15 to R16, R22 to R17, R23 to R18, R16 to R19, R17 to R20, R18 to R21, R19 to R22, R20 to R23, SW2 to SW1, SW1 to SW2
Connections:
- J6 pad 1: (no net) -> Net-(J14-Pad1)
- J6 pad 2: (no net) -> Net-(J14-Pad2)
- J6 pad 3: (no net) -> Net-(J14-Pad3)
- J6 pad 4: (no net) -> GND
- J8 pad 16: Net-(J7-Pad16) -> Net-(J8-Pad16)
- J8 pad 17: Net-(J7-Pad17) -> Net-(J8-Pad17)
- J8 pad 2: Net-(J7-Pad2) -> Net-(J8-Pad2)
- J8 pad 4: Net-(J7-Pad4) -> Net-(J8-Pad4)
- R1 pad 1: Net-(J7-Pad2) -> Net-(J8-Pad2)
- SW1 pad : GND -> (no net)
- SW2 pad A: Net-(R13-Pad2) -> Net-(J8-Pad16)
- SW2 pad B: Net-(R12-Pad2) -> Net-(J8-Pad17)
- SW2 pad C: 3.3V -> GND
- SW2 pad S1: Net-(R14-Pad1) -> Net-(J8-Pad4)
- U1 pad 1: (no net) -> Net-(D1-Pad1)
- U1 pad 2: Net-(D1-Pad1) -> Net-(D1-Pad2)
- U1 pad 3: Net-(D1-Pad2) -> (no net)
- U1 pad 4: (no net) -> Net-(J8-Pad2)
- U1 pad 6: Net-(J7-Pad2) -> 3.3V
Routing:
- net Net-(J8-Pad4): track 0.00 -> 41.5 mm, vias 0 -> 1
- net Net-(J7-Pad2): track 37.6 -> 0.00 mm, vias 1 -> 0
- net Net-(J7-Pad4): track 37.1 -> 0.00 mm, vias 1 -> 0
- net Net-(J8-Pad2): track 0.00 -> 34.8 mm, vias 0 -> 1
- net 3.3V: track 170.2 -> 150.3 mm
- net Net-(J7-Pad17): track 19.5 -> 0.00 mm, vias 1 -> 0
- net Net-(J8-Pad16): track 0.00 -> 19.4 mm
- net Net-(J7-Pad16): track 13.9 -> 0.00 mm, vias 1 -> 0
- net Net-(J8-Pad17): track 0.00 -> 13.8 mm
- net AGND: track 95.2 -> 90.3 mm, vias 4 -> 3
- net Net-(R14-Pad1): track 4.02 -> 0.00 mm
- net Net-(D1-Pad2): track 38.2 -> 42.1 mm
- net Net-(J14-Pad3): track 0.00 -> 3.82 mm
- net Net-(J14-Pad2): track 0.00 -> 3.60 mm
- net Net-(J14-Pad1): track 0.00 -> 3.58 mm
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Other:
- board text added: "11 SEL1/MOSI"
- board text added: "12 " 2 /MISO"
- board text added: "26 FS(Tip)"
- board text added: "5v"
- board text added: "D+"
- board text added: "D-"
- board text added: "Designed by Josh Nishikawa github/joshnishikawa/MomiPlug"
- board text added: "FS(Ring) 15"
- board text added: "SEL0"
- board text added: "SEL1 MOSI0"
- board text added: "SEL2 MISO0"
- board text added: "SEL3 SCK0"
- board text added: "SEL3/SCK0 14"
- board text added: "SIG0 CS0"
- board text added: "SIG0/CS0 20"
- board text added: "SIG1 CS0"
- board text added: "SIG1/CS0 21"
- board text removed: "11 SEL1 / MOSI"
- board text removed: "12 " 2 / MISO"
- board text removed: "26 Footswitch (Tip)"
- board text removed: "Designed by Josh Nishikawa joshnishikawa@gmail.com"
- board text removed: "Footswitch(Ring) 15"
- board text removed: "SEL3 / SCK0 14"
- board text removed: "SIG0 / CS0 20"
- board text removed: "SIG1 / CS0 21"
