File: KiCad/MOMI.sch (KiCad schematic (older format))
At the start: 55 parts, among them J1 Conn_02x04_Male, J10 Conn_01x05_Male, J11 AudioJack4, J12 Conn_01x04_Female, J13 Dual Footswitch, J2 MIDI in, J3 Conn_02x04_Male, J4 MIDI out, J5 JST 1mm (I2C), J6 USB_A, J7 Conn_01x18_Female, J8 Conn_01x18_Female, J9 Expression Pedal, SW1 Encoder_Switch, SW2 SW_SPDT, U1 6N137, U2 MAX1555EZK_T

Commit message: Add KiCad files
Parts:
- removed R12, R13, R14: 10k, R_SMD_3D:R_0805_2012Metric, symbol MOMI-rescue:R-Device
- removed U1: 6N137, Housings_DIP:DIP-8_W7.62mm_Socket, symbol MOMI-rescue:6N137-dk_Optoisolators-Logic-Output
- added J14: Conn_01x03_Male, Pin_Headers:Pin_Header_Straight_1x03_Pitch2.54mm, symbol Connector:Conn_01x03_Male
- added U1: H11L1M, digikey-footprints:DIP-6_W7.62mm, symbol dk_Optoisolators-Logic-Output:H11L1M
- D1: footprint D_SMD_3D:D_0805_2012Metric -> Diodes_ThroughHole:D_A-405_P2.54mm_Vertical_AnodeUp
- D2: value LED -> Green LED
- D3, D4, D8: value LED -> Red LED
- D5: renamed from D7; value LED -> Green LED
- D6: renamed from D5; value LED -> Red LED
- D7: renamed from D6; value LED -> Blue LED
- J2, J4: footprint Connect:SDS-50J -> Conn_Aud_3D:SDS-50J
- renumbered C5 to C2, C2 to C3, C6 to C4, C3 to C5, C4 to C6, J9 to J10, J10 to J11, J11 to J12, J12 to J7, J7 to J8, J8 to J9, R21 to R11, R11 to R12, R15 to R16, R22 to R17, R23 to R18, R16 to R19, R17 to R20, R18 to R21, R19 to R22, R20 to R23, SW2 to SW1, SW1 to SW2
Connections:
- net 3.3V: now also U1.6 (VCC); no longer SW2.C
- net GND: now also J6.4 (GND), SW2.C, U1.5 (GND)
- net at D1.2 (A), J2.5: now also U1.2
- net at SW2.A: now also J8.16 (Pin_16)
- net at SW2.B: now also J8.17 (Pin_17)
- net at SW2.S1: now also J8.4 (Pin_4)
- net at J6.1 (VBUS): now also J14.1 (Pin_1)
- net at J6.2 (D-): now also J14.2 (Pin_2)
- net at J6.3 (D+): now also J14.3 (Pin_3)
- net at J8.2 (Pin_2), R1.1: now also U1.4 (VO)
- net at D1.1 (K), R2.2: now also U1.1
- no-connect marks 11 -> 10
Other:
- moved on the sheet: D1, J1, J2, J3, J4, J5, J6, J7, R1, R2, R3, R4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

Commit message: new pinout for circuit board
Parts:
- removed C1, C6: 10uF, C_SMD_3D:C_0805_2012Metric, symbol MOMI-rescue:CP1-Device
- removed R23: 47k, R_SMD_3D:R_0805_2012Metric, symbol MOMI-rescue:R-Device
- R16: value 47k -> 10k
- U1: symbol dk_Optoisolators-Logic-Output:H11L1M -> MOMI-rescue:H11L1M-dk_Optoisolators-Logic-Output
- U2: symbol dk_PMIC-Battery-Chargers:MAX1555EZK_T -> MOMI-rescue:MAX1555EZK_T-dk_PMIC-Battery-Chargers
Connections:
- net AGND: now also R16.1; no longer J10.RN
- net at J9.1 (Pin_1): now also J10.R, R16.2; no longer R16.1
- net at J9.7 (Pin_7): now also J13.R
- no-connect marks 10 -> 11
Other:
- moved on the sheet: R16
Changed lines of the file:
@@
 Text GLabel 6700 3900 2    50   Input ~ 0
 SEL3&SCK0
-Wire Wire Line
-	6700 5150 6800 5150
-Wire Wire Line
-	7300 5150 7100 5150
-$Comp
-L MOMI-rescue:CP1-Device C1
-U 1 1 5E1743DC
-P 6700 5300
-F 0 "C1" H 6815 5346 50  0000 L CNN
-F 1 "10uF" H 6815 5255 50  0000 L CNN
-F 2 "C_SMD_3D:C_0805_2012Metric" H 6700 5300 50  0001 C CNN
-F 3 "~" H 6700 5300 50  0001 C CNN
-	1    6700 5300
-	-1   0    0    -1
-$EndComp
-$Comp
-L MOMI-rescue:R-Device R16
-U 1 1 5E1743D6
-P 6950 5150
-F 0 "R16" V 7157 5150 50  0000 C CNN
-F 1 "47k" V 7066 5150 50  0000 C CNN
-F 2 "R_SMD_3D:R_0805_2012Metric" V 6880 5150 50  0001 C CNN
-F 3 "~" H 6950 5150 50  0001 C CNN
-	1    6950 5150
-	0    -1   -1   0
-$EndComp
 NoConn ~ 7300 5450
 Text GLabel 7300 5350 0    50   Input ~ 0
@@
 	-1   0    0    -1
 $EndComp
-Wire Wire Line
-	9800 3800 9900 3800
-Wire Wire Line
-	10400 3800 10200 3800
-$Comp
-L MOMI-rescue:R-Device R23
-U 1 1 5E18257F
-P 10050 3800
-F 0 "R23" V 10257 3800 50  0000 C CNN
-F 1 "47k" V 10166 3800 50  0000 C CNN
-F 2 "R_SMD_3D:R_0805_2012Metric" V 9980 3800 50  0001 C CNN
-F 3 "~" H 10050 3800 50  0001 C CNN
-	1    10050 3800
-	0    -1   1    0
-$EndComp
 Text GLabel 10400 3700 0    50   Input ~ 0
 GND
@@
 Wire Wire Line
 	10400 4000 10300 4000
-$Comp
-L MOMI-rescue:CP1-Device C6
-U 1 1 5E182585
-P 9800 3650
-F 0 "C6" H 9915 3696 50  0000 L CNN
-F 1 "10uF" H 9915 3605 50  0000 L CNN
-F 2 "C_SMD_3D:C_0805_2012Metric" H 9800 3650 50  0001 C CNN
-F 3 "~" H 9800 3650 50  0001 C CNN
-	1    9800 3650
-	-1   0    0    1
-$EndComp
-Text GLabel 9800 3500 1    50   Input ~ 0
-GND
 NoConn ~ 10400 3900
-Text GLabel 6700 5450 3    50   Input ~ 0
-AGND
 $Comp
 L MOMI-rescue:AudioJack4-Connector J12
@@
 	0    -1   -1   0
 $EndComp
-Text GLabel 7300 5050 0    50   Input ~ 0
-AGND
-Text GLabel 7300 5250 0    50   Input ~ 0
-AGND
 Text GLabel 1350 5300 2    50   Input ~ 0
 3.3V
@@
 GND
 Wire Wire Line
-	6700 5150 6700 4400
-Connection ~ 6700 5150
-Wire Wire Line
 	8950 4300 6700 4300
 Wire Wire Line
@@
 	10300 4000 10300 6050
 Wire Wire Line
-	9800 3800 6700 3800
-Connection ~ 9800 3800
-Wire Wire Line
 	9600 3700 6700 3700
 Wire Wire Line
@@
 	6700 2350 6700 2700
 $Comp
-L dk_PMIC-Battery-Chargers:MAX1555EZK_T U2
+L MOMI-rescue:MAX1555EZK_T-dk_PMIC-Battery-Chargers U2
 U 1 1 5E1DF4C7
 P 7850 2600
@@
 	2600 2900 2600 4100
 $Comp
-L dk_Optoisolators-Logic-Output:H11L1M U1
+L MOMI-rescue:H11L1M-dk_Optoisolators-Logic-Output U1
 U 1 1 5E2BCD0A
 P 1550 3400
@@
 Wire Wire Line
 	5600 4200 5800 4200
+Wire Wire Line
+	6700 4400 6700 5150
+Wire Wire Line
+	6700 5150 7300 5150
+$Comp
+L MOMI-rescue:R-Device R16
+U 1 1 5E1743D6
+P 6700 5300
+F 0 "R16" V 6907 5300 50  0000 C CNN
+F 1 "10k" V 6816 5300 50  0000 C CNN
+F 2 "R_SMD_3D:R_0805_2012Metric" V 6630 5300 50  0001 C CNN
+F 3 "~" H 6700 5300 50  0001 C CNN
+	1    6700 5300
+	-1   0    0    1
+$EndComp
+Text GLabel 6700 5450 3    50   Input ~ 0
+AGND
+Connection ~ 6700 5150
+Text GLabel 7300 5050 0    50   Input ~ 0
+AGND
+NoConn ~ 7300 5250
+Wire Wire Line
+	6700 3800 10400 3800
 $EndSCHEMATC
